File: talent_dpc200_kicad.sch (KiCad schematic (older format))
At the start: 58 parts, among them CN4 Conn_01x04, CN5 Conn_01x09, CN6 Conn_01x12, U10 D41416C, U11 74LS157, U12 74LS157, U13 TMM4164AP, U14 TMM4164AP, U15 TMM4164AP, U16 TMM4164AP, U17 TMM4164AP, U18 TMM4164AP, U19 TMM4164AP, U20 TMM4164AP, U21 74LS138, U22 74LS32, U28 74LS32, U29 74LS74, U30 74LS367, U31 74LS367, U32 74LS04, U33 74LS00, U34 74LS02, U4 Z80CPU, U5 AY-3-8910, U6 D8255AC-5, U7 TMS9129A, U8 R09256C, U9 D41416C, Y1 10.73MHz

Commit message: Complete schematic up to U23
Parts:
- added C32, C33, C34, C35, C36, C37, C41, C42, C44, C46, C48, C50: ?, symbol Device:C_Small
- added R23, R24, R25, R41: ?, symbol Device:R_Small
- added U23: 74LS74, symbol 74xx:74LS74
- added U24: 74LS153, symbol 74xx:74LS153
- added unit 3 of U28
- added unit 2 of U29
- added U32: 74LS04, symbol 74xx:74LS04
- added unit 2 of U32
- added unit 3 of U32
- added unit 5 of U32
- added unit 6 of U32
- added unit 2 of U33
- added unit 3 of U33
- added unit 2 of U34 (x2)
- added unit 3 of U34
- added unit 4 of U34
- added U37: 74LS07, symbol 74xx:74LS07
- added U41: 74LS374, symbol 74xx:74LS374
Connections:
- net IORQ is gone; now on net ~IORQ~: U31.10 (I4), U4.20 (~IORQ~)
- net RD is gone; now on net ~RD~: U22.4, U28.12, U31.2 (I1), U32.1, U4.21 (~RD~), U8.22 (~OE~/CS1)
- net YS is gone; now on net +12V: RGBJ.5
- net +5V: now also U11.16 (VCC), U12.16 (VCC), U13.8 (VCC), U14.8 (VCC), U15.8 (VCC), U16.8 (VCC), U17.8 (VCC), U18.8 (VCC), U19.8 (VCC), U20.8 (VCC), U21.16 (VCC), U9.9 (VCC), C32.1, C33.1, C34.1, C35.1, C36.1, C37.1, C41.1, C42.1, C44.1, C46.1, C48.1, C50.1, U23.10 (~S), U23.13 (~R), U23.4 (~S)
- net A0: now also U12.2 (I0a), U28.5, U33.1, U34.2, U6.8 (A1), U8.10 (A0)
- net A1: now also U12.5 (I0b), U6.9 (A0), U8.9 (A1)
- net A10: now also U12.13 (I1d), U8.21 (A10)
- net A11: now also U11.3 (I1a), U8.23 (A11)
- net A12: now also U11.6 (I1b), U8.2 (A12)
- net A13: now also U11.10 (I1c), U8.26 (A13)
- net A14: now also U11.14 (I0d), U8.27 (A14)
- net A15: now also U11.13 (I1d)
- net A2: now also U12.11 (I0c), U8.8 (A2)
- net A3: now also U12.14 (I0d), U21.1 (A0), U8.7 (A3)
- net A4: now also U11.2 (I0a), U21.2 (A1), U8.6 (A4)
- net A5: now also U11.5 (I0b), U21.3 (A2), U8.5 (A5)
- net A6: now also U11.11 (I0c), U21.5 (E2), U8.4 (A6)
- net A7: now also U12.3 (I1a), U21.6 (E3), U8.3 (A7)
- net A8: now also U12.6 (I1b), U8.25 (A8)
- net A9: now also U12.10 (I1c), U8.24 (A9)
- net CLK: now also R41.1, U23.11 (C), U23.3 (C), U29.11 (C), U37.12; no longer U31.6 (I3), U4.6 (~CLK~)
- net CPLCLK: now also U22.2
- net D0: now also U17.14 (DOUT), U17.2 (DIN)
- net D1: now also U18.14 (DOUT), U18.2 (DIN)
- net D2: now also U19.14 (DOUT), U19.2 (DIN)
- net D3: now also U20.14 (DOUT), U20.2 (DIN)
- net D4: now also U13.14 (DOUT), U13.2 (DIN)
- net D5: now also U14.14 (DOUT), U14.2 (DIN)
- net D6: now also U15.14 (DOUT), U15.2 (DIN)
- net D7: now also U16.14 (DOUT), U16.2 (DIN)
- net GND: now also U11.15 (E), U11.8 (GND), U12.15 (E), U12.8 (GND), U13.16 (VSS), U14.16 (VSS), U15.16 (VSS), U16.16 (VSS), U17.16 (VSS), U18.16 (VSS), U19.16 (VSS), U20.16 (VSS), U21.8 (GND), C32.2, C33.2, C34.2, C35.2, C36.2, C37.2, C41.2, C42.2, C44.2, C46.2, C48.2, C50.2
- net M1: now also U22.13, U32.4; no longer U31.4 (I2), U4.27 (~M1~)
- net U33:1: no longer U28.5, U33.1, U34.2, U6.9 (A0)
- net ~Y2~: now reaches U21.13 (O2), U28.1, U28.13
- net U28:3: now reaches U28.3, U28.4, U32.9
- net ~Y5~: now reaches U21.10 (O5)
- net ~Y5~: now also U6.6 (~CS~), U33.4
- net ~Y4~: now reaches U21.11 (O4)
- net ~Y4~: now also U34.3, U34.12
- net ~Y3~: now reaches U21.12 (O3)
- net ~Y3~: now also U22.10, U22.5
- net ~Y1~: now reaches U21.14 (O1)
- net ~Y0~: now reaches U21.15 (O0)
- net ~IORQ~+M1: now reaches U21.4 (E1)
- net ~IORQ~+M1: now also U22.11
- net ~Y7~: now reaches U21.7 (O7)
- net ~Y6~: now reaches U21.9 (O6)
- net U28:6: now reaches U28.6, U29.3 (C)
- net U32:8: now reaches U32.8, U33.2
- net U33:3: now reaches U33.3
- net U33:3: now also U41.1 (OE)
- net U34:1: now reaches U34.1
- net U34:1: now also U5.29 (BC1)
- net U23:9: now reaches U5.22 (CLOCK)
- net U23:9: now also U23.9 (Q)
- net U34:13: now reaches U5.27 (BDIR)
- net U34:13: now also U34.13
- net ~RD~: now reaches U6.5 (~RD~)
- net ~CLK~: now reaches U22.3
- net ~CLK~: now also U31.6 (I3), U4.6 (~CLK~), U37.13
- net ~IORQ~: now reaches U22.12
- net at U32.2: now also R25.1
- net MUX: now reaches U11.1 (S)
- net MUX: now also U12.1 (S), U23.2 (D), U34.4
- net L7: now reaches U11.12 (Zd)
- net L7: now also U13.9 (A7), U14.9 (A7), U15.9 (A7), U16.9 (A7), U17.9 (A7), U18.9 (A7), U19.9 (A7), U20.9 (A7)
- net L4: now reaches U11.4 (Za)
- net L4: now also U13.11 (A4), U14.11 (A4), U15.11 (A4), U16.11 (A4), U17.11 (A4), U18.11 (A4), U19.11 (A4), U20.11 (A4)
- net L5: now reaches U11.7 (Zb)
- net L5: now also U13.10 (A5), U14.10 (A5), U15.10 (A5), U16.10 (A5), U17.10 (A5), U18.10 (A5), U19.10 (A5), U20.10 (A5)
- net L6: now reaches U11.9 (Zc)
- net L6: now also U13.13 (A6), U14.13 (A6), U15.13 (A6), U16.13 (A6), U17.13 (A6), U18.13 (A6), U19.13 (A6), U20.13 (A6)
- net L3: now reaches U12.12 (Zd)
- net L3: now also U13.12 (A3), U14.12 (A3), U15.12 (A3), U16.12 (A3), U17.12 (A3), U18.12 (A3), U19.12 (A3), U20.12 (A3)
- net L0: now reaches U12.4 (Za)
- net L0: now also U13.5 (A0), U14.5 (A0), U15.5 (A0), U16.5 (A0), U17.5 (A0), U18.5 (A0), U19.5 (A0), U20.5 (A0)
- net L1: now reaches U12.7 (Zb)
- net L1: now also U13.7 (A1), U14.7 (A1), U15.7 (A1), U16.7 (A1), U17.7 (A1), U18.7 (A1), U19.7 (A1), U20.7 (A1)
- net L2: now reaches U12.9 (Zc)
- net L2: now also U13.6 (A2), U14.6 (A2), U15.6 (A2), U16.6 (A2), U17.6 (A2), U18.6 (A2), U19.6 (A2), U20.6 (A2)
- net ~CAS~: now reaches U13.15 (~CAS~)
- net ~CAS~: now also U14.15 (~CAS~), U15.15 (~CAS~), U16.15 (~CAS~), U17.15 (~CAS~), U18.15 (~CAS~), U19.15 (~CAS~), U20.15 (~CAS~), R23.2
- net ~WRT~: now reaches U13.3 (~WRITE~)
- net ~WRT~: now also U14.3 (~WRITE~), U15.3 (~WRITE~), U16.3 (~WRITE~), U17.3 (~WRITE~), U18.3 (~WRITE~), U19.3 (~WRITE~), U20.3 (~WRITE~), R25.2
- net ~RAS~: now reaches U13.4 (~RAS~)
- net ~RAS~: now also U14.4 (~RAS~), U15.4 (~RAS~), U16.4 (~RAS~), U17.4 (~RAS~), U18.4 (~RAS~), U19.4 (~RAS~), U20.4 (~RAS~), R24.2
- net MREQ renamed ~MREQ~
- net ~MREQ~: now also R24.1
- net RESET renamed ~RESET~
- net ~RESET~: now also U33.10
- net RFSH renamed ~RFSH~
- net WR renamed ~WR~
- new net: R23.1, U23.6 (~Q)
- new net: U23.12 (D), U23.8 (~Q)
- new net: U33.6, U33.9
- new net N.C.?: U23.5 (Q)
- new net U23:3: U37.3
- new net U32:10: U23.1 (~R), U32.10
- new net U33:8: U24.1 (Ea), U24.15 (Eb), U33.5, U33.8
- new net ~M1~: U28.10, U31.4 (I2), U32.3, U4.27 (~M1~)
Other:
- note added: "~Y0~: Not used?"
- note added: "~Y1~: Not used?"
- note added: "~Y2~: Printer?"
- note added: "~Y3~: Video?"
- note added: "~Y4~: Sound?"
- note added: "~Y5~: PPI?"
- note added: "~Y6~: Not used?"
- note added: "~Y7~: Not used?"
- moved on the sheet: C?, D7, R28, R30, TR4, U12, U13, U14, U15, U16, U17, U18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

Commit message: Complete schematic up to U27
Parts:
- added 64K: Jumper_2_Bridged, symbol Jumper:Jumper_2_Bridged
- added C52, C54, C56, C58: ?, symbol Device:C_Small
- added D10: D, symbol Device:D
- added EX1, EX3: Conn_02x25_Odd_Even, symbol Connector_Generic:Conn_02x25_Odd_Even
- added R26, R27, R31: ?, symbol Device:R_Small
- added RELAY: BUSUNG SD 5 V, Relay_THT:Relay_SPDT_SANYOU_SRD_Series_Form_C, symbol Relay:SANYOU_SRD_Form_C
- added TR5: A564, symbol Device:Q_PNP_BCE
- added unit 5 of U22
- added unit 3 of U23
- added U25: 74LS08, symbol 74xx:74LS08
- added U26: 74LS32, symbol 74xx:74LS32
- added U27: 74LS139, symbol 74xx:74LS139
- added unit 4 of U33
Connections:
- net +5V: now also U24.16 (VCC), U29.13 (~R), C52.2, C54.2, C56.2, C58.1, R26.1, R27.1, TR5.3 (E), U22.14 (VCC), U23.14 (VCC), U25.13
- net A14: now also U24.14 (S0), U27.14 (A0)
- net A15: now also U24.2 (S1), U26.12, U27.13 (A1)
- net GND: now also U24.8 (GND), C52.1, C54.1, C56.1, C58.2, D10.2 (A), RELAY.5, U22.7 (GND), U23.7 (GND)
- net N.C.?: now also U4.17 (~NMI~), U26.3, U27.12 (O0); no longer U23.5 (Q)
- net U32:10: now also U29.10 (~S)
- net ~MREQ~: now also U32.13
- net ~RD~: now also U32.1, U26.10, U26.5
- net ~RFSH~: now also U33.13
- net ~INT~+~INT%~: now reaches U4.16 (~INT~)
- net ~INT~+~INT%~: now also U25.3
- net ~WAIT~: now reaches U4.24 (~WAIT~)
- net ~WAIT~: now also U25.6
- net PA3: now reaches U6.1 (PA3)
- net PA3: now also U24.11 (I1b)
- net PC4: now reaches U6.13 (PC4)
- net PC4: now also U25.12
- net PA2: now reaches U6.2 (PA2)
- net PA2: now also U24.5 (I1a)
- net PA1: now reaches U6.3 (PA1)
- net PA1: now also U24.10 (I0b)
- net PA7: now reaches U6.37 (PA7)
- net PA7: now also U24.13 (I3b)
- net PA6: now reaches U6.38 (PA6)
- net PA6: now also U24.3 (I3a)
- net PA5: now reaches U6.39 (PA5)
- net PA5: now also U24.12 (I2b)
- net PA0: now reaches U6.4 (PA0)
- net PA0: now also U24.6 (I0a)
- net PA4: now reaches U6.40 (PA4)
- net PA4: now also U24.4 (I2a)
- net U26:11: now reaches U8.20 (~CE~/CS2)
- net U26:11: now also U26.11
- net ~INT~: now reaches U7.16 (~INT~)
- net ~INT~: now also R26.2, U25.1
- net U28:8: now reaches U28.8
- net U28:8: now also U29.12 (D)
- net U29:8: now reaches U28.9
- net U29:8: now also U29.8 (~Q)
- net at U34.5: now also 64K.2 (B)
- net U24:7: now reaches U24.7 (Za)
- net U24:7: now also U27.2 (A0)
- net U24:9: now reaches U24.9 (Zb)
- net U24:9: now also U27.3 (A1)
- net U33:11: now reaches U32.11
- net U33:11: now also U27.1 (E), U27.15 (E), U33.11
- net MREQ: now reaches U32.12
- net MREQ: now also U33.12
- net U29:9: now reaches U29.9 (Q)
- net U29:9: now also U25.5
- net U23:3: no longer names the net of U37.3
- new net: R31.2, TR5.1 (B)
- new net: D10.1 (K), RELAY.2, TR5.2 (C)
- new net U26:6: EX1.1 (Pin_1), EX3.1 (Pin_1), U25.10, U26.6
- new net U26:8: EX1.2 (Pin_2), EX3.2 (Pin_2), U25.9, U26.8
- new net U27:10: U26.9, U27.10 (O2)
- new net U27:11: U26.4, U27.11 (O1)
- new net U27:9: U26.1, U27.9 (O3)
- new net ~CS12~: EX1.3 (Pin_3), EX3.3 (Pin_3), U25.8
- new net ~INT%~: EX1.8 (Pin_8), EX3.8 (Pin_8), U25.2
- new net ~SLTSL0~: U26.13, U26.2, U27.4 (O0)
- new net ~SLTSL1~: 64K.1 (A), U27.5 (O1)
- new net ~SLTSL2~: EX1.4 (Pin_4), U27.6 (O2)
- new net ~SLTSL3~: EX3.4 (Pin_4), U27.7 (O3)
- new net ~U25:11~: R31.1, U25.11
- new net ~WAIT%~: EX1.7 (Pin_7), EX3.7 (Pin_7), R27.2, U25.4
Other:
- note added: "ROM ENABLE?"
- note added: "TAPE REMOTE PPI?"
- note added: "TAPE REMOTE?"
- note added: "Unconnected pad near"64K"\nsilkscreen marking?"
- note added: "~CS1~?"
- note added: "~CS2~?"
- moved on the sheet: D7, R28, R30, TR4, U29A, U29B, U30, U31
